Commit message: u

File: xacro/cart_effort.xacro (robot description, xacro)
@@ -19,4 +19,7 @@
     </inertial>
   </link>
+  <gazebo reference="slideBar">
+    <material>Gazebo/Orange</material>
+  </gazebo>
 <!-- ****************************************************** cart Link **************************************************************** -->
   <link name="cart">
@@ -35,4 +38,7 @@
     </inertial>
   </link>
+  <gazebo reference="cart">
+    <material>Gazebo/Red</material>
+  </gazebo>
 <!-- ****************************************************** world to slideBar Joint ************************************************** -->
   <joint name="world_to_base" type="fixed">

File: xacro/cart_position.xacro (robot description, xacro)
@@ -19,4 +19,7 @@
     </inertial>
   </link>
+  <gazebo reference="slideBar">
+    <material>Gazebo/Orange</material>
+  </gazebo>
 <!-- ****************************************************** cart Link **************************************************************** -->
   <link name="cart">
@@ -35,4 +38,7 @@
     </inertial>
   </link>
+  <gazebo reference="cart">
+    <material>Gazebo/Red</material>
+  </gazebo>
 <!-- ****************************************************** world to slideBar Joint ************************************************** -->
   <joint name="world_to_base" type="fixed">

File: xacro/cart_velocity.xacro (robot description, xacro)
@@ -19,4 +19,7 @@
     </inertial>
   </link>
+  <gazebo reference="slideBar">
+    <material>Gazebo/Orange</material>
+  </gazebo>
 <!-- ****************************************************** cart Link **************************************************************** -->
   <link name="cart">
@@ -35,4 +38,7 @@
     </inertial>
   </link>
+  <gazebo reference="cart">
+    <material>Gazebo/Red</material>
+  </gazebo>
   <!-- ****************************************************** world to slideBar Joint ************************************************** -->
   <joint name="world_to_base" type="fixed">

File: xacro/gripper_mimic_joint.xacro (robot description, xacro)
@@ -19,4 +19,7 @@
     </inertial>
   </link>
+  <gazebo reference="base">
+    <material>Gazebo/Orange</material>
+  </gazebo>
 <!-- ****************************************************** finger_right Link ******************************************************** -->
   <link name="finger_right">
@@ -35,4 +38,7 @@
     </inertial>
   </link>
+  <gazebo reference="finger_right">
+    <material>Gazebo/Red</material>
+  </gazebo>
 <!-- ****************************************************** finger_left Link ********************************************************* -->
   <link name="finger_left">
@@ -51,4 +57,7 @@
     </inertial>
   </link>
+  <gazebo reference="finger_left">
+    <material>Gazebo/Red</material>
+  </gazebo>
 <!-- ****************************************************** world to base Joint ****************************************************** -->
   <joint name="world_to_base" type="fixed">
